File: free_dry_electrodes_16x3_4cm/free_dry_electrodes_16x3_4cm.kicad_pcb (KiCad board)
At the start: 2 copper layers, 39.6 x 34.3 mm, 27 parts, among them J1 Conn_01x03, J10 Conn_01x03, J11 Conn_01x03, J12 Conn_01x03, J13 Conn_01x03, J14 Conn_01x03, J15 Conn_01x03, J16 Conn_01x03, J17 Conn_01x03, J18 Conn_01x03, J19 Conn_01x03, J2 Conn_01x03, J20 Conn_01x03, J21 Conn_01x03, J22 Conn_01x03, J23 Conn_01x03, J24 Conn_01x03, J3 Conn_01x03, J4 Conn_01x03, J5 Conn_01x03, J6 Conn_01x03, J7 Conn_01x03, J8 Conn_01x03, J9 Conn_01x03

Commit message: Add files via upload
Other:
- board text added: "FreeEEG16-alpha dry electrodes"
- board text removed: "FreeEEG16 Dry Electrodes"
Changed lines of the file:
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@@
     (property "Sheetname" "")
     (fp_text reference "J1" (at 0 3.295) (layer "B.SilkS")
-      (effects (font (size 1 1) (thickness 0.15)) (justify mirror))
+      (effects (font (size 0.762 0.762) (thickness 0.15)) (justify mirror))
     )
     (fp_text value "Conn_01x03" (at 0 -3.295) (layer "B.Fab")
@@
     (property "Sheetname" "")
     (fp_text reference "J4" (at 0 3.295) (layer "B.SilkS")
-      (effects (font (size 1 1) (thickness 0.15)) (justify mirror))
+      (effects (font (size 0.762 0.762) (thickness 0.15)) (justify mirror))
     )
     (fp_text value "Conn_01x03" (at 0 -3.295) (layer "B.Fab")
@@
     (property "Sheetname" "")
     (fp_text reference "J14" (at 0 3.295) (layer "B.SilkS")
-      (effects (font (size 1 1) (thickness 0.15)) (justify mirror))
+      (effects (font (size 0.762 0.762) (thickness 0.15)) (justify mirror))
     )
     (fp_text value "Conn_01x03" (at 0 -3.295) (layer "B.Fab")
@@
     (property "Sheetname" "")
     (fp_text reference "J3" (at 0 3.295) (layer "B.SilkS")
-      (effects (font (size 1 1) (thickness 0.15)) (justify mirror))
+      (effects (font (size 0.762 0.762) (thickness 0.15)) (justify mirror))
     )
     (fp_text value "Conn_01x03" (at 0 -3.295) (layer "B.Fab")
@@
     (property "Sheetname" "")
     (fp_text reference "J10" (at 0 3.295) (layer "B.SilkS")
-      (effects (font (size 1 1) (thickness 0.15)) (justify mirror))
+      (effects (font (size 0.762 0.762) (thickness 0.15)) (justify mirror))
     )
     (fp_text value "Conn_01x03" (at 0 -3.295) (layer "B.Fab")
@@
     (property "Sheetname" "")
     (fp_text reference "J18" (at 0 3.295) (layer "B.SilkS")
-      (effects (font (size 1 1) (thickness 0.15)) (justify mirror))
+      (effects (font (size 0.762 0.762) (thickness 0.15)) (justify mirror))
     )
     (fp_text value "Conn_01x03" (at 0 -3.295) (layer "B.Fab")
@@
     (property "Sheetname" "")
     (fp_text reference "J5" (at 0 3.295) (layer "B.SilkS")
-      (effects (font (size 1 1) (thickness 0.15)) (justify mirror))
+      (effects (font (size 0.762 0.762) (thickness 0.15)) (justify mirror))
     )
     (fp_text value "Conn_01x03" (at 0 -3.295) (layer "B.Fab")
@@
     (property "Sheetname" "")
     (fp_text reference "J2" (at 0 3.295) (layer "B.SilkS")
-      (effects (font (size 1 1) (thickness 0.15)) (justify mirror))
+      (effects (font (size 0.762 0.762) (thickness 0.15)) (justify mirror))
     )
     (fp_text value "Conn_01x03" (at 0 -3.295) (layer "B.Fab")
@@
     (property "Sheetname" "")
     (fp_text reference "J16" (at 0 3.295) (layer "B.SilkS")
-      (effects (font (size 1 1) (thickness 0.15)) (justify mirror))
+      (effects (font (size 0.762 0.762) (thickness 0.15)) (justify mirror))
     )
     (fp_text value "Conn_01x03" (at 0 -3.295) (layer "B.Fab")
@@
     (property "Sheetname" "")
     (fp_text reference "J6" (at 0 3.295) (layer "B.SilkS")
-      (effects (font (size 1 1) (thickness 0.15)) (justify mirror))
+      (effects (font (size 0.762 0.762) (thickness 0.15)) (justify mirror))
     )
     (fp_text value "Conn_01x03" (at 0 -3.295) (layer "B.Fab")
@@
     (property "Sheetname" "")
     (fp_text reference "J12" (at 0 3.295) (layer "B.SilkS")
-      (effects (font (size 1 1) (thickness 0.15)) (justify mirror))
+      (effects (font (size 0.762 0.762) (thickness 0.15)) (justify mirror))
     )
     (fp_text value "Conn_01x03" (at 0 -3.295) (layer "B.Fab")
@@
     (property "Sheetname" "")
     (fp_text reference "J7" (at 0 3.295) (layer "B.SilkS")
-      (effects (font (size 1 1) (thickness 0.15)) (justify mirror))
+      (effects (font (size 0.762 0.762) (thickness 0.15)) (justify mirror))
     )
     (fp_text value "Conn_01x03" (at 0 -3.295) (layer "B.Fab")
@@
     (property "Sheetname" "")
     (fp_text reference "J17" (at 0 3.295) (layer "B.SilkS")
-      (effects (font (size 1 1) (thickness 0.15)) (justify mirror))
+      (effects (font (size 0.762 0.762) (thickness 0.15)) (justify mirror))
     )
     (fp_text value "Conn_01x03" (at 0 -3.295) (layer "B.Fab")
@@
     (property "Sheetname" "")
     (fp_text reference "J8" (at 0 3.295) (layer "B.SilkS")
-      (effects (font (size 1 1) (thickness 0.15)) (justify mirror))
+      (effects (font (size 0.762 0.762) (thickness 0.15)) (justify mirror))
     )
     (fp_text value "Conn_01x03" (at 0 -3.295) (layer "B.Fab")
@@
     (property "Sheetname" "")
     (fp_text reference "J15" (at 0 3.295) (layer "B.SilkS")
-      (effects (font (size 1 1) (thickness 0.15)) (justify mirror))
+      (effects (font (size 0.762 0.762) (thickness 0.15)) (justify mirror))
     )
     (fp_text value "Conn_01x03" (at 0 -3.295) (layer "B.Fab")
@@
     (property "Sheetname" "")
     (fp_text reference "J13" (at 0 3.295) (layer "B.SilkS")
-      (effects (font (size 1 1) (thickness 0.15)) (justify mirror))
+      (effects (font (size 0.762 0.762) (thickness 0.15)) (justify mirror))
     )
     (fp_text value "Conn_01x03" (at 0 -3.295) (layer "B.Fab")
@@
     (property "Sheetname" "")
     (fp_text reference "J9" (at 0 3.295) (layer "B.SilkS")
-      (effects (font (size 1 1) (thickness 0.15)) (justify mirror))
+      (effects (font (size 0.762 0.762) (thickness 0.15)) (justify mirror))
     )
     (fp_text value "Conn_01x03" (at 0.187054 -3.23583) (layer "B.Fab")
@@
     (property "Sheetname" "")
     (fp_text reference "J11" (at 0 3.295) (layer "B.SilkS")
-      (effects (font (size 1 1) (thickness 0.15)) (justify mirror))
+      (effects (font (size 0.762 0.762) (thickness 0.15)) (justify mirror))
     )
     (fp_text value "Conn_01x03" (at 0 -3.295) (layer "B.Fab")
@@
     (effects (font (size 0.75 0.75) (thickness 0.15)) (justify mirror))
   )
-  (gr_text "FreeEEG16\nDry Electrodes" (at 0 0) (layer "F.SilkS")
+  (gr_text "FreeEEG16-alpha\ndry electrodes" (at 0 0) (layer "F.SilkS")
     (effects (font (size 0.75 0.75) (thickness 0.15)))
   )
