File: free_dry_electrodes_16x3_4cm/free_dry_electrodes_16x3_4cm.kicad_sch (KiCad schematic)
At the start: 24 parts, among them J1 Conn_01x03, J10 Conn_01x03, J11 Conn_01x03, J12 Conn_01x03, J13 Conn_01x03, J14 Conn_01x03, J15 Conn_01x03, J16 Conn_01x03, J17 Conn_01x03, J18 Conn_01x03, J19 Conn_01x03, J20 Conn_01x03, J21 Conn_01x03, J22 Conn_01x03, J23 Conn_01x03, J24 Conn_01x03, J3 Conn_01x03, J4 Conn_01x03, J5 Conn_01x03, J6 Conn_01x03, J7 Conn_01x03, J8 Conn_01x03, J9 Conn_01x03

Commit message: Add files via upload
Parts:
- added J25, J26, J27, J? (x6): Conn_02x03_Odd_Even, Connector_PinHeader_1.27mm:PinHeader_2x03_P1.27mm_Vertical, symbol Connector_Generic:Conn_02x03_Odd_Even
- J2: value (none) -> Conn_01x03
Connections:
- net J1: now also J26.2 (Pin_2), J?.1 (Pin_1), J?.2 (Pin_2)
- net J10: now also J25.1 (Pin_1), J?.5 (Pin_5), J?.6 (Pin_6)
- net J11: now also J27.4 (Pin_4), J?.3 (Pin_3), J?.4 (Pin_4)
- net J12: now also J27.1 (Pin_1), J?.5 (Pin_5), J?.6 (Pin_6)
- net J13: now also J25.2 (Pin_2), J?.1 (Pin_1), J?.2 (Pin_2)
- net J14: now also J27.5 (Pin_5), J?.5 (Pin_5), J?.6 (Pin_6)
- net J15: now also J27.3 (Pin_3), J?.1 (Pin_1), J?.2 (Pin_2)
- net J16: now also J27.2 (Pin_2), J?.1 (Pin_1), J?.2 (Pin_2)
- net J17: now also J27.6 (Pin_6), J?.3 (Pin_3), J?.4 (Pin_4)
- net J18: now also J26.6 (Pin_6), J?.3 (Pin_3), J?.4 (Pin_4)
- net J2: now also J26.1 (Pin_1), J?.5 (Pin_5), J?.6 (Pin_6)
- net J3: now also J25.5 (Pin_5), J?.5 (Pin_5), J?.6 (Pin_6)
- net J4: now also J26.3 (Pin_3), J?.1 (Pin_1), J?.2 (Pin_2)
- net J5: now also J25.4 (Pin_4), J?.3 (Pin_3), J?.4 (Pin_4)
- net J6: now also J26.4 (Pin_4), J?.3 (Pin_3), J?.4 (Pin_4)
- net J7: now also J25.3 (Pin_3), J?.1 (Pin_1), J?.2 (Pin_2)
- net J8: now also J25.6 (Pin_6), J?.3 (Pin_3), J?.4 (Pin_4)
- net J9: now also J26.5 (Pin_5), J?.5 (Pin_5), J?.6 (Pin_6)
Other:
- moved on the sheet: J19, J20, J21, J22, J23, J24

Commit message: Add files via upload
Parts:
- gave numbers to parts that had none: 6
Changed lines of the file:
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@@
   (symbol (lib_id "Connector_Generic:Conn_02x03_Odd_Even") (at 152.4 -3.81 0) (unit 1)
     (in_bom yes) (on_board yes) (fields_autoplaced)
-    (property "Reference" "J?" (id 0) (at 153.67 -11.43 0))
+    (property "Reference" "J28" (id 0) (at 153.67 -11.43 0))
     (property "Value" "Conn_02x03_Odd_Even" (id 1) (at 153.67 -8.89 0))
     (property "Footprint" "Connector_PinHeader_1.27mm:PinHeader_2x03_P1.27mm_Vertical" (id 2) (at 152.4 -3.81 0)
@@
   (symbol (lib_id "Connector_Generic:Conn_02x03_Odd_Even") (at 182.88 25.4 0) (unit 1)
     (in_bom yes) (on_board yes)
-    (property "Reference" "J?" (id 0) (at 184.15 17.78 0))
+    (property "Reference" "J33" (id 0) (at 184.15 17.78 0))
     (property "Value" "Conn_02x03_Odd_Even" (id 1) (at 184.15 20.32 0))
     (property "Footprint" "Connector_PinHeader_1.27mm:PinHeader_2x03_P1.27mm_Vertical" (id 2) (at 182.88 25.4 0)
@@
   (symbol (lib_id "Connector_Generic:Conn_02x03_Odd_Even") (at 152.4 26.67 0) (unit 1)
     (in_bom yes) (on_board yes)
-    (property "Reference" "J?" (id 0) (at 153.67 19.05 0))
+    (property "Reference" "J30" (id 0) (at 153.67 19.05 0))
     (property "Value" "Conn_02x03_Odd_Even" (id 1) (at 153.67 21.59 0))
     (property "Footprint" "Connector_PinHeader_1.27mm:PinHeader_2x03_P1.27mm_Vertical" (id 2) (at 152.4 26.67 0)
@@
   (symbol (lib_id "Connector_Generic:Conn_02x03_Odd_Even") (at 182.88 10.16 0) (unit 1)
     (in_bom yes) (on_board yes) (fields_autoplaced)
-    (property "Reference" "J?" (id 0) (at 184.15 2.54 0))
+    (property "Reference" "J32" (id 0) (at 184.15 2.54 0))
     (property "Value" "Conn_02x03_Odd_Even" (id 1) (at 184.15 5.08 0))
     (property "Footprint" "Connector_PinHeader_1.27mm:PinHeader_2x03_P1.27mm_Vertical" (id 2) (at 182.88 10.16 0)
@@
   (symbol (lib_id "Connector_Generic:Conn_02x03_Odd_Even") (at 182.88 -5.08 0) (unit 1)
     (in_bom yes) (on_board yes) (fields_autoplaced)
-    (property "Reference" "J?" (id 0) (at 184.15 -12.7 0))
+    (property "Reference" "J31" (id 0) (at 184.15 -12.7 0))
     (property "Value" "Conn_02x03_Odd_Even" (id 1) (at 184.15 -10.16 0))
     (property "Footprint" "Connector_PinHeader_1.27mm:PinHeader_2x03_P1.27mm_Vertical" (id 2) (at 182.88 -5.08 0)
@@
   (symbol (lib_id "Connector_Generic:Conn_02x03_Odd_Even") (at 152.4 11.43 0) (unit 1)
     (in_bom yes) (on_board yes) (fields_autoplaced)
-    (property "Reference" "J?" (id 0) (at 153.67 3.81 0))
+    (property "Reference" "J29" (id 0) (at 153.67 3.81 0))
     (property "Value" "Conn_02x03_Odd_Even" (id 1) (at 153.67 6.35 0))
     (property "Footprint" "Connector_PinHeader_1.27mm:PinHeader_2x03_P1.27mm_Vertical" (id 2) (at 152.4 11.43 0)
@@
     )
     (path "/13603ae1-712a-48d0-9b7f-9476417e67d2"
-      (reference "J?") (unit 1) (value "Conn_02x03_Odd_Even") (footprint "Connector_PinHeader_1.27mm:PinHeader_2x03_P1.27mm_Vertical")
+      (reference "J28") (unit 1) (value "Conn_02x03_Odd_Even") (footprint "Connector_PinHeader_1.27mm:PinHeader_2x03_P1.27mm_Vertical")
+    )
+    (path "/e2673b7c-e103-49fa-98d5-69b8ba8dd292"
+      (reference "J29") (unit 1) (value "Conn_02x03_Odd_Even") (footprint "Connector_PinHeader_1.27mm:PinHeader_2x03_P1.27mm_Vertical")
+    )
+    (path "/7cea92c9-9703-4eba-a1eb-fed08832ec20"
+      (reference "J30") (unit 1) (value "Conn_02x03_Odd_Even") (footprint "Connector_PinHeader_1.27mm:PinHeader_2x03_P1.27mm_Vertical")
+    )
+    (path "/a7f18a9f-a0be-43eb-b2f0-7c83b416fe20"
+      (reference "J31") (unit 1) (value "Conn_02x03_Odd_Even") (footprint "Connector_PinHeader_1.27mm:PinHeader_2x03_P1.27mm_Vertical")
+    )
+    (path "/8b678575-44ee-4022-9856-b98a338d4a24"
+      (reference "J32") (unit 1) (value "Conn_02x03_Odd_Even") (footprint "Connector_PinHeader_1.27mm:PinHeader_2x03_P1.27mm_Vertical")
     )
     (path "/2582eef6-0eaf-4ecc-b9c6-35ff2de65c52"
-      (reference "J?") (unit 1) (value "Conn_02x03_Odd_Even") (footprint "Connector_PinHeader_1.27mm:PinHeader_2x03_P1.27mm_Vertical")
-    )
-    (path "/7cea92c9-9703-4eba-a1eb-fed08832ec20"
-      (reference "J?") (unit 1) (value "Conn_02x03_Odd_Even") (footprint "Connector_PinHeader_1.27mm:PinHeader_2x03_P1.27mm_Vertical")
-    )
-    (path "/8b678575-44ee-4022-9856-b98a338d4a24"
-      (reference "J?") (unit 1) (value "Conn_02x03_Odd_Even") (footprint "Connector_PinHeader_1.27mm:PinHeader_2x03_P1.27mm_Vertical")
-    )
-    (path "/a7f18a9f-a0be-43eb-b2f0-7c83b416fe20"
-      (reference "J?") (unit 1) (value "Conn_02x03_Odd_Even") (footprint "Connector_PinHeader_1.27mm:PinHeader_2x03_P1.27mm_Vertical")
-    )
-    (path "/e2673b7c-e103-49fa-98d5-69b8ba8dd292"
-      (reference "J?") (unit 1) (value "Conn_02x03_Odd_Even") (footprint "Connector_PinHeader_1.27mm:PinHeader_2x03_P1.27mm_Vertical")
-    )
-  )
+      (reference "J33") (unit 1) (value "Conn_02x03_Odd_Even") (footprint "Connector_PinHeader_1.27mm:PinHeader_2x03_P1.27mm_Vertical")
+    )
+  )
