File: KiCAD/CRYSTAL.kicad_sch (KiCad schematic)
At the start: 1 part, among them U2 FXO-SM7_OSC-SMD7050_short

Commit message: Add files via upload
Parts:
- U2: footprint Oscillator:Oscillator_SMD_ECS_2520MV-xxx-xx-4Pin_2.5x2.0mm -> freeeeg16:Oscillator_SMD_EuroQuartz_XO32-4Pin_3.2x2.5mm_HandSoldering_cut
Changed lines of the file:
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@@
       (effects (font (size 1.524 1.524)))
     )
-    (property "Footprint" "Oscillator:Oscillator_SMD_ECS_2520MV-xxx-xx-4Pin_2.5x2.0mm" (at 135.89 78.74 0)
+    (property "Footprint" "freeeeg16:Oscillator_SMD_EuroQuartz_XO32-4Pin_3.2x2.5mm_HandSoldering_cut" (at 135.89 78.74 0)
       (effects (font (size 1.524 1.524)) hide)
     )

Commit message: Add files via upload
Parts:
- U2: value FXO-SM7_OSC-SMD7050_short -> 8.192MHz; MNP CB3LV-3I-8M1920 -> ECS-2520MVLC-081.92-CN-TR
Changed lines of the file:
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@@
       (effects (font (size 1.524 1.524)))
     )
-    (property "Value" "FXO-SM7_OSC-SMD7050_short" (at 137.16 73.8886 0)
+    (property "Value" "8.192MHz" (at 137.16 73.8886 0)
       (effects (font (size 1.524 1.524)))
     )
@@
       (effects (font (size 1.524 1.524)) hide)
     )
-    (property "MNP" "CB3LV-3I-8M1920" (at 137.16 78.74 0)
+    (property "MNP" "ECS-2520MVLC-081.92-CN-TR" (at 137.16 78.74 0)
       (effects (font (size 1.27 1.27)) hide)
     )
