File: KiCAD/mcu.kicad_sch (KiCad schematic)
At the start: 10 parts, among them U6 STM32F103CBTx, Y1 8.192MHz

Commit message: Add files via upload
Parts:
- C1: MNP (none) -> C0603C475K9PACTU
- C21: value 100nF -> 100n
- U6: MNP (none) -> STM32F103C8T6
Changed lines of the file:
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@@
       (effects (font (size 1.27 1.27)) (justify left))
     )
-    (property "Value" "100nF" (at 75.1332 143.383 0)
+    (property "Value" "100n" (at 75.1332 143.383 0)
       (effects (font (size 1.27 1.27)) (justify left))
     )
@@
       (effects (font (size 1.27 1.27)) (justify left))
     )
-    (property "Value" "100nF" (at 85.2932 143.383 0)
+    (property "Value" "100n" (at 85.2932 143.383 0)
       (effects (font (size 1.27 1.27)) (justify left))
     )
@@
       (effects (font (size 1.27 1.27)) hide)
     )
-    (property "MNP" "" (at 62.23 142.24 0)
+    (property "MNP" "C0603C475K9PACTU" (at 62.23 142.24 0)
       (effects (font (size 1.27 1.27)) hide)
     )
@@
     )
     (property "Datasheet" "http://www.st.com/st-web-ui/static/active/en/resource/technical/document/datasheet/CD00161566.pdf" (at 85.09 77.47 0)
+      (effects (font (size 1.27 1.27)) hide)
+    )
+    (property "MNP" "STM32F103C8T6" (at 85.09 77.47 0)
       (effects (font (size 1.27 1.27)) hide)
     )
@@
       (effects (font (size 1.27 1.27)) (justify left))
     )
-    (property "Value" "100nF" (at 105.6132 143.383 0)
+    (property "Value" "100n" (at 105.6132 143.383 0)
       (effects (font (size 1.27 1.27)) (justify left))
     )
@@
       (effects (font (size 1.27 1.27)) (justify left))
     )
-    (property "Value" "100nF" (at 95.4532 143.383 0)
-      (effects (font (size 1.27 1.27)) (justify left))
-    )
+    (property "Value" "100n" (at 95.4532 143.383 0)
+      (effects (font (size 1.27 1.27)) (justify left))
+    )
