File: KiCAD/radio.kicad_sch (KiCad schematic)
At the start: 3 parts, among them U9 ESP32-C3-WROOM-02

Commit message: Add files via upload
Parts:
- U9: symbol Espressif:ESP32-C3-WROOM-02 -> FreeEEG16-alpha-adc_mcu:ESP32-C3-WROOM-02_allpins
Connections:
- net GND renamed 19_GND
- net 19_GND: no longer U9.9 (GND)
- new net 9_GND: U9.9 (GND)
Changed lines of the file:
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@@
+    (stroke (width 0) (type default))
+  )
+  (wire (pts (xy 95.25 77.47) (xy 97.79 77.47))
     (stroke (width 0) (type default))
   )
@@
   (wire (pts (xy 41.91 69.85) (xy 39.37 69.85))
     (stroke (width 0) (type default))
+  )
+  (hierarchical_label "9_GND" (shape input) (at 97.79 77.47 0) (fields_autoplaced)
+    (effects (font (size 1.27 1.27)) (justify left))
   )
   (hierarchical_label "1_3V3" (shape input) (at 91.44 96.52 90) (fields_autoplaced)
@@
     (effects (font (size 1.27 1.27)) (justify left))
   )
-  (symbol (lib_id "Espressif:ESP32-C3-WROOM-02") (at 69.85 57.15 0) (unit 1)
+  (symbol (lib_id "FreeEEG16-alpha-adc_mcu:ESP32-C3-WROOM-02_allpins") (at 69.85 57.15 0) (unit 1)
     (in_bom yes) (on_board yes) (dnp no) (fields_autoplaced)
     (property "Reference" "U9" (at 69.85 26.67 0)

Commit message: Add files via upload
Parts:
- C1: MNP (none) -> GRM188R60J106ME47D
- C21: value 100nF -> 100n
- U9: MNP (none) -> ESP32-C3-WROOM-02U-N4
Changed lines of the file:
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@@
+      (effects (font (size 1.27 1.27)) hide)
+    )
+    (property "MNP" "ESP32-C3-WROOM-02U-N4" (at 69.85 57.15 0)
       (effects (font (size 1.27 1.27)) hide)
     )
@@
       (effects (font (size 1.27 1.27)) hide)
     )
-    (property "MNP" "" (at 76.2 101.6 0)
+    (property "MNP" "GRM188R60J106ME47D" (at 76.2 101.6 0)
       (effects (font (size 1.27 1.27)) hide)
     )
@@
       (effects (font (size 1.27 1.27)) (justify left))
     )
-    (property "Value" "100nF" (at 89.1032 102.743 0)
+    (property "Value" "100n" (at 89.1032 102.743 0)
       (effects (font (size 1.27 1.27)) (justify left))
     )
