File: KiCAD/vref.kicad_sch (KiCad schematic)
At the start: 7 parts, among them U1 REF2025

Commit message: Add files via upload
Parts:
- C23, C25: MNP CL05B104KO5NNNC -> (none)
- C24: footprint Capacitor_SMD:C_0603_1608Metric -> Capacitor_SMD:C_0402_1005Metric; MNP CL05B104KO5NNNC -> CL05A105KO5NNNC
Changed lines of the file:
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@@
       (effects (font (size 1.27 1.27)) (justify left))
     )
-    (property "Footprint" "Capacitor_SMD:C_0603_1608Metric" (at 97.79 99.06 0)
+    (property "Footprint" "Capacitor_SMD:C_0402_1005Metric" (at 97.79 99.06 0)
       (effects (font (size 1.27 1.27)) hide)
     )
@@
       (effects (font (size 1.27 1.27)) hide)
     )
-    (property "MNP" "CL05B104KO5NNNC" (at 97.79 99.06 0)
+    (property "MNP" "CL05A105KO5NNNC" (at 97.79 99.06 0)
       (effects (font (size 1.27 1.27)) hide)
     )
@@
       (effects (font (size 1.27 1.27)) hide)
     )
-    (property "MNP" "CL05B104KO5NNNC" (at 87.63 99.06 0)
+    (property "MNP" "" (at 87.63 99.06 0)
       (effects (font (size 1.27 1.27)) hide)
     )
@@
       (effects (font (size 1.27 1.27)) hide)
     )
-    (property "MNP" "CL05B104KO5NNNC" (at 107.95 99.06 0)
+    (property "MNP" "" (at 107.95 99.06 0)
       (effects (font (size 1.27 1.27)) hide)
     )
