File: KiCAD/3V3.kicad_sch (KiCad schematic)
At the start: 4 parts, among them U10 AMS1117-3.3

Commit message: Add files via upload
Parts:
- removed U11: ~, symbol FreeEEG32-ads131-rescue:LP5907-lp5907
- C16, C17: MNP GRM188R71A225KE15D -> GRM21BR60J226ME39L
- U10: MNP (none) -> TLV1117-33IDCY
Changed lines of the file:
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@@
       (effects (font (size 1.27 1.27)) hide)
     )
-    (property "MNP" "GRM188R71A225KE15D" (at 102.87 68.58 0)
+    (property "MNP" "GRM21BR60J226ME39L" (at 102.87 68.58 0)
       (effects (font (size 1.27 1.27)) hide)
     )
@@
         (path "/909b030b-fa1a-4fe8-b1ee-422b4d9e23cf/befe1c4c-9a73-480a-bd63-7ff39e5aa340"
           (reference "C17") (unit 1)
-        )
-      )
-    )
-  )
-  (symbol (lib_id "FreeEEG32-ads131-rescue:LP5907-lp5907") (at 83.82 59.69 0) (unit 1)
-    (in_bom yes) (on_board yes) (dnp no)
-    (property "Reference" "U11" (at 83.82 48.1838 0)
-      (effects (font (size 1.524 1.524)))
-    )
-    (property "Value" "~" (at 83.82 50.8762 0)
-      (effects (font (size 1.524 1.524)))
-    )
-    (property "Footprint" "" (at 83.82 53.5686 0)
-      (effects (font (size 1.524 1.524)))
-    )
-    (property "Datasheet" "" (at 83.82 59.69 0)
-      (effects (font (size 1.524 1.524)))
-    )
-    (property "MNP" "LP5907QMFX-3.3Q1" (at 83.82 59.69 0)
-      (effects (font (size 1.27 1.27)) hide)
-    )
-    (property "Manufacturer" "Texas Instruments" (at 83.82 59.69 0)
-      (effects (font (size 1.27 1.27)) hide)
-    )
-    (pin "1")
-    (pin "2")
-    (pin "3")
-    (pin "4")
-    (pin "5")
-    (instances
-      (project "freeeeg16-alpha"
-        (path "/909b030b-fa1a-4fe8-b1ee-422b4d9e23cf/befe1c4c-9a73-480a-bd63-7ff39e5aa340"
-          (reference "U11") (unit 1)
         )
       )
@@
     )
     (property "Datasheet" "http://www.advanced-monolithic.com/pdf/ds1117.pdf" (at 85.09 31.75 0)
+      (effects (font (size 1.27 1.27)) hide)
+    )
+    (property "MNP" "TLV1117-33IDCY" (at 82.55 25.4 0)
       (effects (font (size 1.27 1.27)) hide)
     )
@@
       (effects (font (size 1.27 1.27)) hide)
     )
-    (property "MNP" "GRM188R71A225KE15D" (at 60.96 67.31 0)
+    (property "MNP" "GRM21BR60J226ME39L" (at 60.96 67.31 0)
       (effects (font (size 1.27 1.27)) hide)
     )
