File: KiCAD/ADC2_ads131.kicad_sch (KiCad schematic)
At the start: 5 parts, among them U3 ADS131M08IPBSR

Commit message: Add files via upload
Parts:
- C21: value 100nF -> 100n
- C6: value 220nF -> 220n
Changed lines of the file:
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@@
       (effects (font (size 1.27 1.27)) (justify left))
     )
-    (property "Value" "100nF" (at 86.5632 126.873 0)
+    (property "Value" "100n" (at 86.5632 126.873 0)
       (effects (font (size 1.27 1.27)) (justify left))
     )
@@
       (effects (font (size 1.27 1.27)) (justify left))
     )
-    (property "Value" "220nF" (at 86.5632 106.553 0)
+    (property "Value" "220n" (at 86.5632 106.553 0)
       (effects (font (size 1.27 1.27)) (justify left))
     )
