File: KiCAD/vref1.kicad_sch (KiCad schematic)
At the start: 5 parts, among them U13 REF35125

Commit message: Add files via upload
Parts:
- C27: footprint Capacitor_SMD:C_0603_1608Metric -> Capacitor_SMD:C_0402_1005Metric; MNP CL05B104KO5NNNC -> CL05A105KO5NNNC
- C29: MNP CL05B104KO5NNNC -> GRM188R60J106ME47D
- U13: MNP (none) -> REF35120QDBVR
Changed lines of the file:
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@@
       (effects (font (size 1.27 1.27)) (justify left))
     )
-    (property "Footprint" "Capacitor_SMD:C_0603_1608Metric" (at 86.36 83.82 0)
+    (property "Footprint" "Capacitor_SMD:C_0402_1005Metric" (at 86.36 83.82 0)
       (effects (font (size 1.27 1.27)) hide)
     )
@@
       (effects (font (size 1.27 1.27)) hide)
     )
-    (property "MNP" "CL05B104KO5NNNC" (at 86.36 83.82 0)
+    (property "MNP" "CL05A105KO5NNNC" (at 86.36 83.82 0)
       (effects (font (size 1.27 1.27)) hide)
     )
@@
     (property "Datasheet" "" (at 86.36 39.37 0)
       (effects (font (size 1.524 1.524)))
+    )
+    (property "MNP" "REF35120QDBVR" (at 86.36 39.37 0)
+      (effects (font (size 1.27 1.27)) hide)
     )
     (pin "1")
@@
       (effects (font (size 1.27 1.27)) hide)
     )
-    (property "MNP" "CL05B104KO5NNNC" (at 96.52 83.82 0)
+    (property "MNP" "GRM188R60J106ME47D" (at 96.52 83.82 0)
       (effects (font (size 1.27 1.27)) hide)
     )
