File: KiCAD/freeeeg16-alpha.kicad_pcb (KiCad board)
At the start: 4 copper layers, 39.6 x 34.3 mm, 60 parts, among them J1 Conn_02x03_Odd_Even, J28 Conn_02x03_Odd_Even, J29 Conn_02x03_Odd_Even, J30 Conn_02x03_Odd_Even, J31 Conn_02x03_Odd_Even, J32 Conn_02x03_Odd_Even, J33 Conn_02x03_Odd_Even, J5 Conn_01x07, J6 Conn_01x06, SW1 SW_Push, SW2 SW_Push, SW3 SW_Push, SW4 SW_Push, U10 AMS1117-3.3, U13 REF35125, U2 FXO-SM7_OSC-SMD7050_short, U3 ADS131M08IPBSR, U4 LP5907, U5 LP5907, U6 STM32F103CBTx, U7 LP5907, U8 ADS131M08IPBSR, U9 ESP32-C3-WROOM-02

Commit message: Add files via upload
Parts:
- C38, R4: moved to B.Cu
- J5: footprint Connector_Molex:Molex_PicoBlade_53398-0771_1x07-1MP_P1.25mm_Vertical -> freeeeg16:Molex_PicoBlade_53398-0871_1x08-1MP_P1.25mm_Vertical_cut
- U2: footprint Oscillator:Oscillator_SMD_ECS_2520MV-xxx-xx-4Pin_2.5x2.0mm -> freeeeg16:Oscillator_SMD_EuroQuartz_XO32-4Pin_3.2x2.5mm_HandSoldering_cut
- moved C38 7.58 mm to (-0.03, -14.0)
- moved U2 0.63 mm to (0.00, -13.6), turned to -90 degrees
- moved R4 0.25 mm to (0.00, -15.2)
- moved C37 0.13 mm to (-7.11, -8.00)
Connections:
- J5 pad 6: MCU_37_PA14_SYS_JTCK-SWCLK -> MCU_39_PB3_SYS_JTDO-TRACESWO
- U6 pad 42: /MCU/42_PB6 -> ACC_13_SCL
- U6 pad 43: /MCU/43_PB7 -> ACC_14_SDA
- U9 pad 10: /RADIO/10_GPIO10 -> ACC_13_SCL
- U9 pad 15: /RADIO/15_GPIO3 -> ACC_14_SDA
Routing:
- net ACC_14_SDA: track 0.00 -> 16.3 mm, vias 0 -> 1
- net MCU_18_PB0_ADC1_SYNC/RESET: track 53.2 -> 37.6 mm
- net ACC_13_SCL: track 0.00 -> 7.24 mm, vias 0 -> 1
- net 3V3_2_GND: track 135.2 -> 141.5 mm
- net ACC_5_VDDIO: track 92.5 -> 95.7 mm, vias 7 -> 6
- net MCU_37_PA14_SYS_JTCK-SWCLK: track 4.71 -> 1.60 mm
- net MCU_39_PB3_SYS_JTDO-TRACESWO: track 0.00 -> 2.85 mm, vias 0 -> 1
- net ADC2_21_DIN: track 14.6 -> 16.6 mm
- net ADC2_17_CS: track 10.7 -> 12.6 mm
- net RADIO_16_GPIO2: track 7.92 -> 6.12 mm
- net MCU_5_PDO0_RCC_OSC_IN: track 35.6 -> 37.1 mm
- net ADC1_16_SYNC/RESET: track 34.8 -> 33.4 mm
- net RADIO_8_GPIO9: track 43.3 -> 44.6 mm
- net CRYSTAL_3_OUT: track 5.05 -> 6.28 mm
- net 3V3_5_OUT: track 59.3 -> 60.5 mm
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
Commit message: Add files via upload
Parts:
- removed SW1, SW2, SW3, SW4: SW_Push, Button_Switch_SMD:SW_SPST_B3U-1000P-B
- added J2: Conn_01x03, Connector_PinHeader_1.27mm:PinHeader_1x03_P1.27mm_Vertical, F.Cu at (-12.3, 1.10)
- added J3: Conn_01x03, Connector_PinHeader_1.27mm:PinHeader_1x03_P1.27mm_Vertical, F.Cu at (12.3, 1.10)
- added R10: 0, Resistor_SMD:R_0402_1005Metric, B.Cu at (10.7, 1.40)
- added R8: 0, Resistor_SMD:R_0402_1005Metric, B.Cu at (-10.6, 1.45)
- C38: moved to F.Cu
- C41: moved to B.Cu
- moved C41 21.0 mm to (-6.50, 8.94), turned to 135 degrees
- moved C38 14.4 mm to (-10.4, -4.01), turned to -120 degrees
- moved C39 2.70 mm to (-10.2, 1.42)
- moved C20 1.96 mm to (-5.08, 10.3)
- moved R5 1.84 mm to (5.71, 9.47)
- moved C5 0.16 mm to (1.04, -3.58)
- moved R4 0.13 mm to (0.00, -15.4)
Connections:
- J28 pad 3: ADC1_32_AIN1P -> /J18
- J28 pad 4: ADC1_32_AIN1P -> /J18
- J28 pad 5: ADC1_01_AIN2P -> ADC1_32_AIN1P
- J28 pad 6: ADC1_01_AIN2P -> ADC1_32_AIN1P
- J30 pad 1: ADC1_04_AIN3P -> ADC1_01_AIN2P
- J30 pad 2: ADC1_04_AIN3P -> ADC1_01_AIN2P
- J30 pad 3: ADC1_05_AIN4P -> ADC1_04_AIN3P
- J30 pad 4: ADC1_05_AIN4P -> ADC1_04_AIN3P
- J30 pad 5: ADC1_08_AIN5P -> ADC1_05_AIN4P
- J30 pad 6: ADC1_08_AIN5P -> ADC1_05_AIN4P
- J31 pad 1: ADC2_01_AIN2P -> ADC2_04_AIN3P
- J31 pad 2: ADC2_01_AIN2P -> ADC2_04_AIN3P
- J31 pad 3: ADC2_04_AIN3P -> /J17
- J31 pad 4: ADC2_04_AIN3P -> /J17
- J32 pad 1: ADC1_09_AIN6P -> ADC1_08_AIN5P
- J32 pad 2: ADC1_09_AIN6P -> ADC1_08_AIN5P
- J32 pad 3: ADC1_12_AIN7P -> ADC1_09_AIN6P
- J32 pad 4: ADC1_12_AIN7P -> ADC1_09_AIN6P
- J32 pad 5: 3V3_2_GND -> ADC1_12_AIN7P
- J32 pad 6: 3V3_2_GND -> ADC1_12_AIN7P
- J33 pad 1: ADC1_02_AIN2N -> ADC2_29_AIN0P
- J33 pad 2: ADC1_02_AIN2N -> ADC2_29_AIN0P
- J33 pad 3: ADC2_29_AIN0P -> ADC2_32_AIN1P
- J33 pad 4: ADC2_29_AIN0P -> ADC2_32_AIN1P
- J33 pad 5: ADC2_32_AIN1P -> ADC2_01_AIN2P
- J33 pad 6: ADC2_32_AIN1P -> ADC2_01_AIN2P
Routing:
- net RADIO_8_GPIO9: track 44.6 -> 5.27 mm, vias 2 -> 1
- net ADC1_09_AIN6P: track 14.1 -> 47.1 mm, vias 0 -> 1
- net /J18: track 0.00 -> 20.2 mm
- net ADC1_02_AIN2N: track 71.4 -> 56.1 mm, vias 2 -> 3
- net ADC1_08_AIN5P: track 6.72 -> 16.0 mm, vias 0 -> 1
- net ADC2_01_AIN2P: track 6.72 -> 15.3 mm, vias 0 -> 1
- net /J17: track 0.00 -> 8.24 mm
- net MCU_7_NRST: track 13.7 -> 5.85 mm
- net 3V3_2_GND: track 141.5 -> 133.9 mm
- net ADC1_26_DVDD: track 50.8 -> 44.6 mm
- net ACC_5_VDDIO: track 95.7 -> 91.4 mm
- net ADC1_12_AIN7P: track 14.9 -> 17.0 mm, vias 0 -> 1
- net ADC1_01_AIN2P: track 10.8 -> 9.17 mm
- net ADC2_29_AIN0P: track 14.7 -> 16.3 mm, vias 0 -> 1
- net ADC1_14_REFIN: track 44.8 -> 46.3 mm
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
Commit message: Add files via upload
Parts:
- C12, C6: value 220nF -> 220n
- C21, C22, C33, C34, C35, C36, C38: value 100nF -> 100n
- C27: footprint Capacitor_SMD:C_0603_1608Metric -> Capacitor_SMD:C_0402_1005Metric
- J5: value Conn_01x07 -> Conn_01x08
- U2: value FXO-SM7_OSC-SMD7050_short -> 8.192MHz
Routing:
- net 3V3_2_GND: track 133.9 -> 145.2 mm
- net ADC1_15_AVDD: track 59.7 -> 67.8 mm
- net 3V3_1_IN: track 80.5 -> 87.1 mm
- net 3V3_5_OUT: track 60.1 -> 66.1 mm
- net ADC1_14_REFIN: track 46.3 -> 45.0 mm
- net ACC_5_VDDIO: track 91.4 -> 90.4 mm
- net ADC1_16_SYNC/RESET: track 34.4 -> 35.0 mm
- net MCU_18_PB0_ADC1_SYNC/RESET: track 37.7 -> 38.3 mm

Commit message: Add files via upload
Routing:
- net MCU_5_PDO0_RCC_OSC_IN: track 37.1 -> 36.3 mm
- net ADC2_17_CS: track 13.0 -> 12.4 mm
- net ADC2_21_DIN: track 16.6 -> 17.1 mm

Commit message: Add files via upload
Parts:
- added C40: 100n, Capacitor_SMD:C_0402_1005Metric, B.Cu at (12.6, 10.1)
- added C43: 10u DNP, Capacitor_SMD:C_0603_1608Metric, F.Cu at (13.3, 10.4)
- added R11: 0, Resistor_SMD:R_0402_1005Metric, F.Cu at (16.1, 6.58)
- added R12: 0 DNP, Resistor_SMD:R_0402_1005Metric, B.Cu at (13.3, 10.5)
- U13: value REF35125 -> MAX6070AAUT12
- moved C26 1.32 mm to (17.2, 9.91)
- moved C27 0.65 mm to (18.0, 10.4)
Connections:
- J6 pad 4: ADC1_14_REFIN -> VREF1_6_VREF
- U13 pad 1: 3V3_2_GND -> /vref2/1_FILTER
- U13 pad 5: /vref1/5_NR -> Net-(U13-OUTS)
Routing:
- net Net-(U13-OUTS): track 0.00 -> 11.1 mm
- net ADC1_14_REFIN: track 45.0 -> 51.9 mm
- net /vref2/1_FILTER: track 0.00 -> 3.90 mm, vias 0 -> 1
- net ADC2_17_CS: track 12.4 -> 9.95 mm
- net 3V3_2_GND: track 145.2 -> 147.3 mm, vias 16 -> 17
- net 3V3_1_IN: track 87.1 -> 86.0 mm
- net ADC1_15_AVDD: track 67.8 -> 67.0 mm
- net MCU_18_PB0_ADC1_SYNC/RESET: track 38.3 -> 37.8 mm

Commit message: Add files via upload
Parts:
- added R13: 10k, Resistor_SMD:R_0402_1005Metric, F.Cu at (-10.5, 2.82)
- C39: value 100n -> 1u
- moved C35 4.13 mm to (4.11, 10.7), turned to 0 degrees
- moved R7 1.07 mm to (-10.5, 4.24), turned to 165 degrees
- moved C39 0.36 mm to (-10.5, 1.65), turned to -15 degrees
Connections:
- J6 pad 4: VREF1_6_VREF -> ADC1_14_REFIN
Routing:
- net 3V3_2_GND: track 147.3 -> 144.8 mm, vias 17 -> 18
- net RADIO_2_EN: track 6.00 -> 7.67 mm
- net ACC_5_VDDIO: track 90.4 -> 92.0 mm
- net RADIO_7_GPIO8: track 1.31 -> 2.26 mm
- net MCU_5_PDO0_RCC_OSC_IN: track 36.3 -> 36.9 mm
- net MCU_44_BOOT0: track 3.81 -> 3.26 mm
- net (no net): track 0.00 -> 0.04 mm, vias 0 -> 2
