File: KiCAD/freeeeg16-alpha.kicad_sch (KiCad schematic)
At the start: 23 parts, among them J1 Conn_02x03_Odd_Even, J28 Conn_02x03_Odd_Even, J29 Conn_02x03_Odd_Even, J30 Conn_02x03_Odd_Even, J31 Conn_02x03_Odd_Even, J32 Conn_02x03_Odd_Even, J33 Conn_02x03_Odd_Even, J5 Conn_01x07, J6 Conn_01x06, SW1 SW_Push, SW2 SW_Push, SW3 SW_Push, SW4 SW_Push

Commit message: Add files via upload
Parts:
- J5: footprint Connector_Molex:Molex_PicoBlade_53398-0771_1x07-1MP_P1.25mm_Vertical -> freeeeg16:Molex_PicoBlade_53398-0871_1x08-1MP_P1.25mm_Vertical_cut
Connections:
- net MCU_37_PA14_SYS_JTCK-SWCLK: now also J5.8 (Pin_8); no longer J5.6 (Pin_6)
- net MCU_39_PB3_SYS_JTDO-TRACESWO: now also J5.6 (Pin_6); no longer J5.8 (Pin_8)
Other:
- sheet RADIO ports: added 9_GND; removed none

Commit message: Add files via upload
Parts:
- added J2, J3: Conn_01x03, Connector_PinHeader_1.27mm:PinHeader_1x03_P1.27mm_Vertical, symbol Connector_Generic:Conn_01x03
- added R10, R8: 0, Resistor_SMD:R_0402_1005Metric, symbol FreeEEG32-ads131-rescue:R_Small-Device
Connections:
- net 3V3_2_GND: now also J2.1 (Pin_1), R8.2; no longer J32.5 (Pin_5), J32.6 (Pin_6)
- net ADC1_01_AIN2P: now also J30.1 (Pin_1), J30.2 (Pin_2); no longer J28.5 (Pin_5), J28.6 (Pin_6)
- net ADC1_02_AIN2N: now also J3.1 (Pin_1), R10.2; no longer J33.1 (Pin_1), J33.2 (Pin_2)
- net ADC1_04_AIN3P: now also J30.3 (Pin_3), J30.4 (Pin_4); no longer J30.1 (Pin_1), J30.2 (Pin_2)
- net ADC1_05_AIN4P: now also J30.5 (Pin_5), J30.6 (Pin_6); no longer J30.3 (Pin_3), J30.4 (Pin_4)
- net ADC1_08_AIN5P: now also J32.1 (Pin_1), J32.2 (Pin_2); no longer J30.5 (Pin_5), J30.6 (Pin_6)
- net ADC1_09_AIN6P: now also J32.3 (Pin_3), J32.4 (Pin_4), J2.3 (Pin_3), J3.3 (Pin_3); no longer J32.1 (Pin_1), J32.2 (Pin_2)
- net ADC1_12_AIN7P: now also J32.5 (Pin_5), J32.6 (Pin_6); no longer J32.3 (Pin_3), J32.4 (Pin_4)
- net ADC1_32_AIN1P: now also J28.5 (Pin_5), J28.6 (Pin_6); no longer J28.3 (Pin_3), J28.4 (Pin_4)
- net ADC2_01_AIN2P: now also J33.5 (Pin_5), J33.6 (Pin_6); no longer J31.1 (Pin_1), J31.2 (Pin_2)
- net ADC2_04_AIN3P: now also J31.1 (Pin_1), J31.2 (Pin_2); no longer J31.3 (Pin_3), J31.4 (Pin_4)
- net ADC2_29_AIN0P: now also J33.1 (Pin_1), J33.2 (Pin_2); no longer J33.3 (Pin_3), J33.4 (Pin_4)
- net ADC2_32_AIN1P: now also J33.3 (Pin_3), J33.4 (Pin_4); no longer J33.5 (Pin_5), J33.6 (Pin_6)
- new net J17: J3.2 (Pin_2), J31.3 (Pin_3), J31.4 (Pin_4), R10.1
- new net J18: J2.2 (Pin_2), J28.3 (Pin_3), J28.4 (Pin_4), R8.1

Commit message: Add files via upload
Parts:
- J1, J2, J3: MNP (none) -> 20021111-00006T1LF
- J28, J29, J30, J31, J32, J33: MNP (none) -> 20021311-00006T4LF
- J5: value Conn_01x07 -> Conn_01x08; MNP (none) -> 53398-0871
- J6: MNP (none) -> 53398-0671
- R7, R9: MNP RC0402JR-074K7L -> RC0402JR-0710KL
Changed lines of the file:
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@@
       (effects (font (size 1.27 1.27)) hide)
     )
-    (property "MNP" "RC0402JR-074K7L" (at 160.02 92.71 0)
+    (property "MNP" "RC0402JR-0710KL" (at 160.02 92.71 0)
       (effects (font (size 1.27 1.27)) hide)
     )
@@
       (effects (font (size 1.27 1.27)) hide)
     )
+    (property "MNP" "20021311-00006T4LF" (at 95.25 101.6 0)
+      (effects (font (size 1.27 1.27)) hide)
+    )
     (pin "1")
     (pin "2")
@@
       (effects (font (size 1.27 1.27)) hide)
     )
+    (property "MNP" "20021311-00006T4LF" (at 120.65 116.84 0)
+      (effects (font (size 1.27 1.27)) hide)
+    )
     (pin "1")
     (pin "2")
@@
       (effects (font (size 1.27 1.27)) hide)
     )
+    (property "MNP" "20021111-00006T1LF" (at 73.66 134.62 0)
+      (effects (font (size 1.27 1.27)) hide)
+    )
     (pin "1")
     (pin "2")
@@
     )
     (property "Datasheet" "~" (at 95.25 132.08 0)
+      (effects (font (size 1.27 1.27)) hide)
+    )
+    (property "MNP" "20021311-00006T4LF" (at 95.25 132.08 0)
       (effects (font (size 1.27 1.27)) hide)
     )
@@
       (effects (font (size 1.27 1.27)) hide)
     )
-    (property "MNP" "RC0402JR-074K7L" (at 163.83 90.17 0)
+    (property "MNP" "RC0402JR-0710KL" (at 163.83 90.17 0)
       (effects (font (size 1.27 1.27)) hide)
     )
@@
     )
     (property "Datasheet" "~" (at 93.98 146.05 0)
+      (effects (font (size 1.27 1.27)) hide)
+    )
+    (property "MNP" "20021111-00006T1LF" (at 93.98 146.05 0)
       (effects (font (size 1.27 1.27)) hide)
     )
@@
       (effects (font (size 1.27 1.27)) hide)
     )
+    (property "MNP" "20021311-00006T4LF" (at 95.25 116.84 0)
+      (effects (font (size 1.27 1.27)) hide)
+    )
     (pin "1")
     (pin "2")
@@
       (effects (font (size 1.27 1.27)) (justify left))
     )
-    (property "Value" "Conn_01x07" (at 180.34 138.4299 0)
+    (property "Value" "Conn_01x08" (at 180.34 138.4299 0)
       (effects (font (size 1.27 1.27)) (justify left))
     )
@@
     )
     (property "Datasheet" "~" (at 177.8 137.16 0)
+      (effects (font (size 1.27 1.27)) hide)
+    )
+    (property "MNP" "53398-0871" (at 177.8 137.16 0)
       (effects (font (size 1.27 1.27)) hide)
     )
@@
       (effects (font (size 1.27 1.27)) hide)
     )
+    (property "MNP" "53398-0671" (at 172.72 157.48 0)
+      (effects (font (size 1.27 1.27)) hide)
+    )
     (pin "1")
     (pin "2")
@@
       (effects (font (size 1.27 1.27)) hide)
     )
+    (property "MNP" "20021111-00006T1LF" (at 34.29 134.62 0)
+      (effects (font (size 1.27 1.27)) hide)
+    )
     (pin "1")
     (pin "2")
@@
     )
     (property "Datasheet" "~" (at 120.65 132.08 0)
+      (effects (font (size 1.27 1.27)) hide)
+    )
+    (property "MNP" "20021311-00006T4LF" (at 120.65 132.08 0)
       (effects (font (size 1.27 1.27)) hide)
     )
@@
       (effects (font (size 1.27 1.27)) hide)
     )
+    (property "MNP" "20021311-00006T4LF" (at 120.65 101.6 0)
+      (effects (font (size 1.27 1.27)) hide)
+    )

Commit message: Add files via upload
Other:
- moved on the sheet: C20, C39, C41, J1, J2, J3, J5, J6, R1, R10, R2, R4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

Commit message: Add files via upload
Connections:
- net ADC1_14_REFIN: no longer J6.4 (Pin_4)
- new net VREF1_6_VREF: J6.4 (Pin_4)
Other:
- removed sheet vref
- removed sheet vref1
- added sheet vref2 (vref2.kicad_sch)
- moved on the sheet: C20, C39, C41, J2, J3, R10, R5, R8, SW1, SW2, SW3, SW4

Commit message: Add files via upload
Parts:
- added R13: 10k, Resistor_SMD:R_0402_1005Metric, symbol FreeEEG32-ads131-rescue:R_Small-Device
- C39: value 100n -> 1u; MNP CL05B104KO5NNNC -> CL05A105KO5NNNC
Connections:
- net VREF1_6_VREF is gone; now on net ADC1_14_REFIN: J6.4 (Pin_4)
- net 3V3_5_OUT: now also R13.2
- net RADIO_2_EN: now also R13.1
Other:
- moved on the sheet: C20, C39, C41, R5, SW1, SW2, SW3, SW4
