File: KiCAD/vref2.kicad_sch (KiCad schematic)
At the start: 9 parts, among them U13 MAX6070AAUT12

Commit message: Add files via upload
Parts:
- renumbered C26 to C40, C29 to C43
Changed lines of the file:
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@@
   (symbol (lib_id "FreeEEG32-ads131-rescue:C_Small-Device") (at 121.92 39.37 270) (unit 1)
     (in_bom yes) (on_board yes) (dnp no)
-    (property "Reference" "C29" (at 123.0884 41.7068 0)
+    (property "Reference" "C43" (at 123.0884 41.7068 0)
       (effects (font (size 1.27 1.27)) (justify left))
     )
@@
   (symbol (lib_id "FreeEEG32-ads131-rescue:C_Small-Device") (at 62.23 63.5 270) (unit 1)
     (in_bom yes) (on_board yes) (dnp no)
-    (property "Reference" "C26" (at 63.3984 65.8368 0)
-      (effects (font (size 1.27 1.27)) (justify left))
-    )
+    (property "Reference" "C40" (at 63.3984 65.8368 0)
+      (effects (font (size 1.27 1.27)) (justify left))
+    )
